File: shoe_box_pcb.kicad_sch (KiCad schematic)
At the start: 0 parts

Commit message: updated mcu and added connectors
Parts:
- added D1: D, Diode_THT:D_DO-35_SOD27_P7.62mm_Horizontal, symbol Device:D
- added J1: Conn_01x02_Pin, Module:ST_Morpho_Connector_144_STLink, symbol Connector:Conn_01x02_Pin
- added J2: Conn_01x07, symbol Connector_Generic:Conn_01x07
- added U1: ATmega328-P, Package_DIP:DIP-28_W7.62mm, symbol MCU_Microchip_ATmega:ATmega328-P
Connections:
- new net +3.3V: J2.5 (Pin_5)
- new net +5V: U1.20 (AVCC), U1.7 (VCC)
- new net BTN: J1.1 (Pin_1), U1.4 (PD2)
- new net GND: D1.2 (A), J1.2 (Pin_2), J2.7 (Pin_7), U1.22 (GND), U1.8 (GND)
- new net MISO: J2.4 (Pin_4), U1.18 (PB4)
- new net MOSI: J2.3 (Pin_3), U1.17 (PB3)
- new net RELAY: D1.1 (K), U1.13 (PD7)
- new net RST: J2.6 (Pin_6), U1.14 (PB0)
- new net SCK: J2.2 (Pin_2), U1.19 (PB5)
- new net SDA: J2.1 (Pin_1), U1.16 (PB2)
- no-connect marks 0 -> 17
